File: triple-effect-order-switching-board.kicad_sch (KiCad schematic)
At the start: 7 parts, among them J1 Conn_01x08, J2 Conn_01x08, SW1 SW_3PDT, SW2 SW_3PDT, SW3 SW_3PDT

Commit message: finished board
Parts:
- removed D1, D2: LED, bca-footprints:LED_D5.0mm, symbol Device:LED
- added SW4: SW_3PDT, bca-footprints:SW_Foot_3PDT, symbol BCA Symbol Library:SW_3PDT
- added SW5: SW_3PDT, bca-footprints:SW_Toggle_3PDT_SolderLug, symbol BCA Symbol Library:SW_3PDT
- J1, J2: footprint bca-footprints:Pin_Header_Straight_1x06_Pitch2.54mm -> bca-footprints:Pin_Header_Straight_1x08_Pitch2.54mm; symbol Connector_Generic:Conn_01x06 -> Connector_Generic:Conn_01x08
Connections:
- net Earth: now also SW2.3 (C), SW3.6 (C), SW4.3 (C); no longer SW2.9 (C), SW3.3 (C)
- net in0: now also SW2.1 (A), SW5.4 (A), SW5.9 (C); no longer SW1.1 (A), SW1.9 (C), SW2.7 (A)
- net in1: now also SW1.9 (C), SW3.3 (C), SW3.4 (A); no longer SW1.3 (C), SW3.1 (A), SW3.6 (C)
- net input_jack: now also SW5.5 (B); no longer SW1.2 (B)
- net led0: now also J1.5 (Pin_5), SW2.8 (B); no longer SW2.2 (B)
- net led1: now also J2.2 (Pin_2)
- net out0: now also SW5.2 (B); no longer SW1.5 (B)
- net out1: now also SW1.2 (B), SW3.2 (B); no longer SW1.8 (B), SW3.5 (B)
- net output_jack: now also J2.8 (Pin_8), SW5.3 (C), SW5.7 (A); no longer J2.5 (Pin_5), SW1.6 (C), SW1.7 (A)
- net return1: now also J1.8 (Pin_8), SW3.1 (A); no longer J2.4 (Pin_4), SW3.4 (A)
- net send0: now also SW2.2 (B); no longer SW2.8 (B)
- net send1: now also J1.7 (Pin_7), SW3.5 (B); no longer J2.3 (Pin_3), SW3.2 (B)
- net v0: now also SW2.7 (A); no longer SW2.1 (A)
- net v1: now also J2.3 (Pin_3); no longer J2.6 (Pin_6)
- new net in2: SW1.1 (A), SW1.6 (C), SW4.1 (A), SW4.6 (C)
- new net led2: J2.6 (Pin_6), SW4.8 (B)
- new net os_in: SW1.5 (B), SW5.1 (A), SW5.6 (C)
- new net os_out: SW1.3 (C), SW1.7 (A), SW5.8 (B)
- new net out2: SW1.8 (B), SW4.5 (B)
- new net return2: J2.5 (Pin_5), SW4.4 (A)
- new net send2: J2.4 (Pin_4), SW4.2 (B)
- new net v2: J2.7 (Pin_7), SW4.7 (A)
Other:
- note added: "Bypass C"
- note added: "Pre/Post Switch"
- moved on the sheet: SW1A, SW1B, SW1C, SW2A, SW2B, SW2C, SW3A, SW3B, SW3C
